File: EEG_ADS1299_5.kicad_pcb (KiCad board)
At the start: 2 copper layers, 49.6 x 21.2 mm, 90 parts, among them IC1 ADS1299, P1 CONN_2, P2 CONN_2, P3 CONN_1, P4 CONN_1, P5 CONN_01X08, P6 CONN_2, U1 TPS2294x, U2 TPS61222, U3 NRF528XX-QFAA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

Commit message: Done with adjustments. Needs final revision before shipping
Other:
- board text added: "+5V"
- board text added: "VBAT"
- board text removed: "+Vin (4.5→5.5V)"
- board text removed: "BAT"
- board text removed: "USB CHG"
Changed lines of the file:
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@@
     (links 244)
     (no_connects 0)
-    (area 258.206428 111.37 320.907143 145.345)
+    (area 264.418 111.37 320.907143 139.410001)
     (thickness 1.6)
     (drawings 41)
@@
     (mod_text_size 1 1)
     (mod_text_width 0.15)
-    (pad_size 0.7 0.24)
-    (pad_drill 0)
+    (pad_size 1.524 1.524)
+    (pad_drill 1.016)
     (pad_to_mask_clearance 0.015)
     (aux_axis_origin 0 0)
@@
     )
   )
+  (gr_text GND (at 271.7 114.95 90) (layer F.SilkS)
+    (effects (font (size 0.75 0.75) (thickness 0.1)))
+  )
   (gr_line (start 315.47 134.17) (end 315.48 134.17) (angle 90) (layer Edge.Cuts) (width 0.1))
   (gr_line (start 315.47 112.99) (end 315.47 134.17) (angle 90) (layer Edge.Cuts) (width 0.1))
@@
   (gr_line (start 278.11 127.26) (end 278.11 128.06) (angle 90) (layer F.SilkS) (width 0.2))
   (gr_line (start 278.78 127.7) (end 279.78 127.7) (angle 90) (layer F.SilkS) (width 0.2))
-  (gr_text "USB CHG" (at 262.71 135.44) (layer F.SilkS)
+  (gr_text VBAT (at 269.28 117.77 90) (layer F.SilkS)
     (effects (font (size 0.75 0.75) (thickness 0.1)))
   )
-  (gr_text "+Vin (4.5→5.5V)" (at 261.935 138.41) (layer F.SilkS)
-    (effects (font (size 0.6 0.6) (thickness 0.1)))
-  )
-  (gr_text GND (at 264.785 133.235) (layer F.SilkS)
+  (gr_text GND (at 267.35 122.19) (layer F.SilkS)
     (effects (font (size 0.75 0.75) (thickness 0.1)))
   )
   (gr_line (start 311.08 125.5) (end 311.1 125.5) (angle 90) (layer Edge.Cuts) (width 0.1))
   (gr_circle (center 285.8125 117.6125) (end 285.6125 117.5125) (layer F.SilkS) (width 0.2))
-  (gr_text + (at 306.02 130.55) (layer F.SilkS)
+  (gr_text + (at 311.54 117.31) (layer F.SilkS)
     (effects (font (size 0.74 0.75) (thickness 0.1)))
   )
-  (gr_text — (at 308.34 130.48) (layer F.SilkS)
+  (gr_text — (at 314.29 117.42) (layer F.SilkS)
     (effects (font (size 0.74 0.75) (thickness 0.1)))
   )
-  (gr_text CH4 (at 310.26 140.11 270) (layer F.SilkS)
+  (gr_text CH4 (at 309.79 126.72 270) (layer F.SilkS)
     (effects (font (size 0.74 0.75) (thickness 0.1)))
   )
-  (gr_text CH3 (at 310.24 137.59 270) (layer F.SilkS)
+  (gr_text CH3 (at 309.91 124.28 270) (layer F.SilkS)
     (effects (font (size 0.74 0.75) (thickness 0.1)))
   )
-  (gr_text I/O (at 300.31 128.9) (layer F.SilkS)
+  (gr_text I/O (at 274.8 123.95) (layer F.SilkS)
     (effects (font (size 0.7 0.7) (thickness 0.1)))
   )
@@
   (gr_line (start 272.4 125.5) (end 272.4 132) (angle 90) (layer F.SilkS) (width 0.2))
   (gr_line (start 265.9 125.5) (end 272.4 125.5) (angle 90) (layer F.SilkS) (width 0.2))
-  (gr_text ADS1299-x (at 315.06 142.26 180) (layer F.SilkS)
+  (gr_text ADS1299-x (at 297.99 124.82 180) (layer F.SilkS)
     (effects (font (size 1 1) (thickness 0.125)))
   )
@@
     (effects (font (size 1 1) (thickness 0.125)))
   )
-  (gr_text "BIAS/\nGND" (at 308.93 143.72 90) (layer F.SilkS)
+  (gr_text "BIAS/\nGND" (at 309.46 130.33 90) (layer F.SilkS)
     (effects (font (size 0.74 0.75) (thickness 0.1)))
   )
-  (gr_text CH2 (at 310.24 135.01 270) (layer F.SilkS)
+  (gr_text CH2 (at 309.94 121.88 270) (layer F.SilkS)
     (effects (font (size 0.74 0.75) (thickness 0.1)))
   )
-  (gr_text SRB1 (at 306.24 126.84) (layer F.SilkS)
+  (gr_text SRB1 (at 310.55 114.99 90) (layer F.SilkS)
     (effects (font (size 0.74 0.75) (thickness 0.1)))
   )
-  (gr_text CH1 (at 310.24 132.6 270) (layer F.SilkS)
+  (gr_text CH1 (at 309.91 119.29 270) (layer F.SilkS)
     (effects (font (size 0.74 0.75) (thickness 0.1)))
   )
@@
     (effects (font (size 1.5 1.5) (thickness 0.3)))
   )
-  (gr_text CLK (at 302.78 128.85) (layer F.SilkS)
+  (gr_text CLK (at 277.37 123.93) (layer F.SilkS)
     (effects (font (size 0.7 0.7) (thickness 0.1)))
   )
-  (gr_text BAT (at 261.58 134.29) (layer F.SilkS)
+  (gr_text +5V (at 267.21 113.61) (layer F.SilkS)
     (effects (font (size 0.75 0.75) (thickness 0.1)))
   )
@@
     (polygon
       (pts
-        (xy 315.51 139.41) (xy 265.91 139.41) (xy 265.91 132) (xy 272.41 132) (xy 272.41 123.3)
+        (xy 315.51 139.41) (xy 265.91 139.41) (xy 265.91 134.2) (xy 272.41 134.2) (xy 272.41 123.3)
         (xy 265.9 123.3) (xy 265.9 111.37) (xy 315.51 111.37)
       )
@@
     (polygon
       (pts
-        (xy 315.51 139.41) (xy 265.91 139.41) (xy 265.91 132) (xy 272.41 132) (xy 272.41 123.3)
+        (xy 315.51 139.41) (xy 265.91 139.41) (xy 265.91 134.2) (xy 272.41 134.2) (xy 272.41 123.3)
         (xy 265.9 123.3) (xy 265.9 111.37) (xy 315.51 111.37)
       )
