File: EEG_ADS1299_2.sch (KiCad schematic (older format))
At the start: 89 parts, among them IC1 ADS1299, P1 CONN_2, P2 CONN_2, P3 CONN_1, P4 CONN_1, P5 CONN_01X08, P6 CONN_2, U1 TPS2294x, U2 TPS61222, U3 NRF528XX-QFAA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

Commit message: Huge update. Rough draft of device with battery management.
Parts:
- added J1: USB_OTG, symbol USB_OTG
- R19, R20: value 10k -> 1M
Connections:
- net labels added: N.C.
- wire segments 368 -> 379
Other:
- note added: "FOR RECHARGING: \nusing Amphenol FCI 10103594-0001LF"
- note removed: "FOR RECHARGING:"
- note removed: "Remove switch??"
- moved on the sheet: P3, P4
Changed lines of the file:
@@
 L VCC #PWR04
 U 1 1 58A71443
-P 10000 1350
-F 0 "#PWR04" H 10000 1450 30  0001 C CNN
-F 1 "VCC" H 10000 1450 30  0000 C CNN
-F 2 "" H 10000 1350 60  0000 C CNN
-F 3 "" H 10000 1350 60  0000 C CNN
-	1    10000 1350
+P 1100 7850
+F 0 "#PWR04" H 1100 7950 30  0001 C CNN
+F 1 "VCC" H 1100 7950 30  0000 C CNN
+F 2 "" H 1100 7850 60  0000 C CNN
+F 3 "" H 1100 7850 60  0000 C CNN
+	1    1100 7850
 	1    0    0    -1
 $EndComp
@@
 	1    0    0    -1
 $EndComp
-Text Notes 8250 1350 0    60   ~ 0
+Text Notes -650 7850 0    60   ~ 0
 Power Regulation Circuit
 Text Label 12600 11450 0    60   ~ 0
@@
 Text Label 6800 7450 2    60   ~ 0
 IN1
-Text Label 4250 7700 2    60   ~ 0
+Text Label 7000 6500 2    60   ~ 0
 SRB1
 Text GLabel 29100 4700 3    60   Input ~ 0
@@
 	1    0    0    -1
 $EndComp
-Text Label 4300 7350 2    60   ~ 0
+Text Label 7050 6150 2    60   ~ 0
 BIASIN
 Text Label 23500 6300 1    60   ~ 0
@@
 Text Notes 15900 3100 0    60   ~ 0
 Apparently supposed to be 3.3µH????\nSee TI forumns/ WEBENCH
-Text Notes 10150 2100 0    60   ~ 0
-Remove switch??
 $Comp
 L C C14
@@
 L CONN_1 P4
 U 1 1 58B800EE
-P 3400 7350
-F 0 "P4" V 3350 7350 40  0000 C CNN
-F 1 "CONN_1" V 3450 7350 40  0000 C CNN
-F 2 "Pin_Headers:Pin_Header_Straight_1x01_Pitch2.54mm" H 3400 7350 60  0001 C CNN
-F 3 "" H 3400 7350 60  0000 C CNN
-	1    3400 7350
+P 6150 6150
+F 0 "P4" V 6100 6150 40  0000 C CNN
+F 1 "CONN_1" V 6200 6150 40  0000 C CNN
+F 2 "Pin_Headers:Pin_Header_Straight_1x01_Pitch2.54mm" H 6150 6150 60  0001 C CNN
+F 3 "" H 6150 6150 60  0000 C CNN
+	1    6150 6150
 	-1   0    0    1
 $EndComp
@@
 L CONN_1 P3
 U 1 1 591A6E5B
-P 3400 7700
-F 0 "P3" V 3350 7700 40  0000 C CNN
-F 1 "CONN_1" V 3450 7700 40  0000 C CNN
-F 2 "Pin_Headers:Pin_Header_Straight_1x01_Pitch2.54mm" H 3400 7700 60  0001 C CNN
-F 3 "" H 3400 7700 60  0000 C CNN
-	1    3400 7700
+P 6150 6500
+F 0 "P3" V 6100 6500 40  0000 C CNN
+F 1 "CONN_1" V 6200 6500 40  0000 C CNN
+F 2 "Pin_Headers:Pin_Header_Straight_1x01_Pitch2.54mm" H 6150 6500 60  0001 C CNN
+F 3 "" H 6150 6500 60  0000 C CNN
+	1    6150 6500
 	-1   0    0    1
 $EndComp
@@
 	1    0    0    -1
 $EndComp
-Text Label 22150 5650 2    60   ~ 0
-LED2
-Text Label 22150 5750 2    60   ~ 0
-LED3
 Text GLabel 21450 4450 3    60   Input ~ 0
 DGND
@@
 Text Label 13050 2500 0    60   ~ 0
 SYS_LOAD
-Text Label 11600 1600 0    60   ~ 0
+Text Label 2700 8100 0    60   ~ 0
 BATT_VOLTAGE
 $Comp
@@
 P 9650 18500
 F 0 "R19" V 9730 18500 50  0000 C CNN
-F 1 "10k" V 9650 18500 50  0000 C CNN
+F 1 "1M" V 9650 18500 50  0000 C CNN
 F 2 "Resistors_SMD:R_0402" V 9580 18500 50  0001 C CNN
 F 3 "" H 9650 18500 50  0000 C CNN
@@
 P 10000 18700
 F 0 "R20" V 10080 18700 50  0000 C CNN
-F 1 "10k" V 10000 18700 50  0000 C CNN
+F 1 "1M" V 10000 18700 50  0000 C CNN
 F 2 "Resistors_SMD:R_0402" V 9930 18700 50  0001 C CNN
 F 3 "" H 10000 18700 50  0000 C CNN
@@
 Text Notes 10850 19000 0    60   ~ 0
 CTRL pin. Low disables VINSW, high enables VINSW
-Text Label 20350 4750 0    60   ~ 0
+Text Label 19550 5750 0    60   ~ 0
 BATT_ADC_AIN
 Text Notes 4650 11650 0    60   ~ 0
@@
 	1    0    0    -1
 $EndComp
-Text Label 20350 4900 0    60   ~ 0
+Text Label 19550 5650 0    60   ~ 0
 GPIO_CTRL_PWR_ON
 Text Notes 6950 15000 0    60   ~ 0
 We're using TPS610981
-Text Label 20350 5050 0    60   ~ 0
+Text Label 19650 6050 0    60   ~ 0
 GPIO_OVERCURRENT
+Text Label 20350 5400 0    60   ~ 0
+GPIO_ISET
+Text Label 20350 5300 0    60   ~ 0
+GPIO_TTDM_BAT_EN
+Text GLabel 13900 3750 1    60   Input ~ 0
+DGND
+Text Label 4100 6850 0    60   ~ 0
+DC+INPUT
+Text Notes 3400 6500 0    60   ~ 0
+FOR RECHARGING: \nusing Amphenol FCI 10103594-0001LF
+$Comp
+L USB_OTG J1
+U 1 1 59BAF4BC
+P 3550 7050
+F 0 "J1" H 3350 7500 50  0000 L CNN
+F 1 "USB_OTG" H 3350 7400 50  0000 L CNN
+F 2 "" H 3700 7000 50  0001 C CNN
+F 3 "" H 3700 7000 50  0001 C CNN
+	1    3550 7050
+	1    0    0    -1
+$EndComp
+Text Label 4550 7150 0    60   ~ 0
+SWDIO
+Text Label 4450 7000 0    60   ~ 0
+SWDCLK
+Text Label 4450 7350 0    60   ~ 0
+N.C.
+$Comp
+L GND-RESCUE-emg_circuit_2_ext_amp #PWR015
+U 1 1 59BB26FA
+P 4100 7700
+F 0 "#PWR015" H 4100 7700 30  0001 C CNN
+F 1 "GND" H 4100 7630 30  0001 C CNN
+F 2 "" H 4100 7700 60  0000 C CNN
+F 3 "" H 4100 7700 60  0000 C CNN
+	1    4100 7700
+	1    0    0    -1
+$EndComp
+Text Label 24350 6450 0    60   ~ 0
+LED2
+Text Label 25350 4800 2    60   ~ 0
+LED3
+$Comp
+L CONN_2 P6
+U 1 1 59BE4BF7
+P 3450 8500
+F 0 "P6" V 3400 8500 40  0000 C CNN
+F 1 "CONN_2" V 3500 8500 40  0000 C CNN
+F 2 "Pin_Headers:Pin_Header_Straight_1x02_Pitch2.54mm" H 3450 8500 60  0001 C CNN
+F 3 "" H 3450 8500 60  0000 C CNN
+	1    3450 8500
+	-1   0    0    -1
+$EndComp
+$Comp
+L GND-RESCUE-emg_circuit_2_ext_amp #PWR016
+U 1 1 59BE4F90
+P 4300 8700
+F 0 "#PWR016" H 4300 8700 30  0001 C CNN
+F 1 "GND" H 4300 8630 30  0001 C CNN
+F 2 "" H 4300 8700 60  0000 C CNN
+F 3 "" H 4300 8700 60  0000 C CNN
+	1    4300 8700
+	1    0    0    -1
+$EndComp
+Text Label 4250 8400 0    60   ~ 0
+DC+INPUT
 Wire Wire Line
 	23800 5700 23800 6850
@@
 	6300 6750 6800 6750
 Wire Wire Line
-	3750 7700 4250 7700
+	6500 6500 7000 6500
 Wire Notes Line
 	500  6100 5350 6100
 Wire Notes Line
-	5350 6100 5350 7750
+	5350 6100 5350 8250
 Wire Wire Line
 	23700 5700 23700 6300
@@
 	18550 1100 8050 1100
 Wire Wire Line
-	10000 1350 10000 1600
-Wire Wire Line
-	10000 1600 11600 1600
+	1100 7850 1100 8100
+Wire Wire Line
+	1100 8100 2700 8100
 Wire Wire Line
 	18000 7800 18000 7700
@@
 	15150 12250 15350 12250
 Wire Wire Line
-	3750 7350 4300 7350
+	6500 6150 7050 6150
 Wire Wire Line
 	13800 6350 13800 6600
@@
 Wire Notes Line
 	17450 2900 15850 2900
-Wire Notes Line
-	9900 1150 9900 2150
-Wire Notes Line
-	9900 2150 12100 2150
-Wire Notes Line
-	12100 2150 12100 1100
 Wire Notes Line
 	12100 1100 9900 1100
@@
 Connection ~ 6650 19300
 Wire Wire Line
-	22450 4300 22650 4300
-Wire Wire Line
-	22500 4400 22650 4400
-Wire Wire Line
-	22450 4300 22450 4750
-Wire Wire Line
-	22450 4750 20350 4750
-Wire Wire Line
-	22500 4400 22500 4900
-Wire Wire Line
-	22500 4900 20350 4900
-Wire Wire Line
-	22650 4500 22550 4500
-Wire Wire Line
-	22550 4500 22550 5050
-Wire Wire Line
-	22550 5050 20350 5050
-Wire Wire Line
-	22150 5650 22600 5650
-Wire Wire Line
-	22600 5650 22600 5000
-Wire Wire Line
-	22600 5000 22650 5000
-Wire Wire Line
-	22650 5100 22650 5750
-Wire Wire Line
-	22650 5750 22150 5750
-Wire Wire Line
-	22650 4700 21950 4700
-Wire Wire Line
-	21950 4700 21950 5300
-Wire Wire Line
 	21950 5300 20350 5300
 Wire Wire Line
-	22650 4800 22050 4800
-Wire Wire Line
-	22050 4800 22050 5400
-Wire Wire Line
 	22050 5400 20350 5400
-Text Label 20350 5300 0    60   ~ 0
-GPIO_ISET
-Text Label 20350 5400 0    60   ~ 0
-GPIO_TTDM_BAT_EN
-Text GLabel 13900 3750 1    60   Input ~ 0
-DGND
-$Comp
-L CONN_2 P6
-U 1 1 59BD8B22
-P 2050 8500
-F 0 "P6" V 2000 8500 40  0000 C CNN
-F 1 "CONN_2" V 2100 8500 40  0000 C CNN
-F 2 "Pin_Headers:Pin_Header_Straight_1x02_Pitch2.54mm" H 2050 8500 60  0001 C CNN
-F 3 "" H 2050 8500 60  0000 C CNN
-	1    2050 8500
-	-1   0    0    -1
-$EndComp
-Wire Wire Line
-	2400 8400 2900 8400
-Text Label 2900 8400 0    60   ~ 0
-DC+INPUT
-Text Notes 2300 8200 0    60   ~ 0
-FOR RECHARGING:
-Wire Wire Line
-	2400 8600 2900 8600
-$Comp
-L GND-RESCUE-emg_circuit_2_ext_amp #PWR015
-U 1 1 59BD9771
-P 2900 8700
-F 0 "#PWR015" H 2900 8700 30  0001 C CNN
-F 1 "GND" H 2900 8630 30  0001 C CNN
-F 2 "" H 2900 8700 60  0000 C CNN
-F 3 "" H 2900 8700 60  0000 C CNN
-	1    2900 8700
-	1    0    0    -1
-$EndComp
-Wire Wire Line
-	2900 8600 2900 8700
+Wire Wire Line
+	4100 6850 3850 6850
+Wire Wire Line
+	3850 7050 4100 7050
+Wire Wire Line
+	3850 7150 4100 7150
+Wire Wire Line
+	3850 7250 4100 7250
+Wire Wire Line
+	3550 7450 3550 7550
+Wire Wire Line
+	3450 7550 4100 7550
+Wire Wire Line
+	4100 7550 4100 7700
+Wire Wire Line
+	3450 7550 3450 7450
+Connection ~ 3550 7550
+Wire Notes Line
+	5700 5850 5700 7650
+Wire Notes Line
+	5700 7650 7450 7650
+Wire Notes Line
+	7450 7650 7450 5850
+Wire Notes Line
+	7450 5850 5700 5850
+Wire Notes Line
+	5350 8250 550  8250
+Wire Wire Line
+	25050 4700 25350 4700
+Wire Wire Line
+	25050 4800 25350 4800
+Wire Wire Line
+	22650 4300 22450 4300
+Wire Wire Line
+	22450 4300 22450 4550
+Wire Wire Line
+	22450 4550 21950 4550
+Wire Wire Line
+	21950 4550 21950 5300
+Wire Wire Line
+	22050 5400 22050 4600
+Wire Wire Line
+	22050 4600 22550 4600
+Wire Wire Line
+	22550 4600 22550 4400
+Wire Wire Line
+	22550 4400 22650 4400
+Wire Wire Line
+	22650 4500 22200 4500
+Wire Wire Line
+	22200 4500 22200 5650
+Wire Wire Line
+	22200 5650 19550 5650
+Wire Wire Line
+	19550 5750 22250 5750
+Wire Wire Line
+	22250 5750 22250 4600
+Wire Wire Line
+	22250 4600 22650 4600
+Wire Wire Line
+	22300 5850 19550 5850
+Wire Wire Line
+	3800 8600 4300 8600
+Wire Wire Line
+	4300 8600 4300 8700
+Wire Wire Line
+	3800 8400 4250 8400
+Wire Wire Line
+	22650 4700 22300 4700
+Wire Wire Line
+	22300 4700 22300 5850
+Wire Wire Line
+	24100 5700 24100 6450
+Wire Wire Line
+	24100 6450 24350 6450
 $EndSCHEMATC

Commit message: Updated battery management design v2 complete.
Parts:
- removed L3: 15nH, Inductors_SMD:L_0402, symbol INDUCTOR
- removed L4: 10uH, Inductors_SMD:L_0603, symbol INDUCTOR
- C10, C22, C23: footprint Capacitors_SMD:C_0603 -> Capacitors_SMD:C_0402
Connections:
- net labels added: DEC4
- wire segments 379 -> 388
- no-connect marks 16 -> 17
Other:
- note added: "TPS22941 is the one we will use"

Commit message: Done with adjustments. Needs final revision before shipping
Connections:
- wire segments 388 -> 383
Changed lines of the file:
@@
 	22350 4100 22350 4300
 Wire Wire Line
-	23900 2950 25050 2950
-Wire Wire Line
 	23800 2850 25050 2850
-Wire Wire Line
-	25050 2750 23700 2750
 Wire Wire Line
 	23600 3300 23600 2750
@@
 	23800 2850 23800 3300
 Wire Wire Line
-	23900 2950 23900 3300
-Wire Wire Line
-	24000 3300 24000 3050
-Wire Wire Line
-	24100 3300 24100 3050
-Wire Wire Line
 	3800 8400 4250 8400

Commit message: Final version, v4.
Parts:
- added P10, P7, P8, P9: CONN_01X02, symbol CONN_01X02
- J1: symbol USB_OTG -> USB_OTG-RESCUE-EEG_ADS1299_2
Connections:
- wire segments 383 -> 395
Other:
- moved on the sheet: P5
Changed lines of the file:
@@
 This network will need to be tuned
 $Comp
-L GND-RESCUE-emg_circuit_2_ext_amp #PWR01
+L GND-RESCUE-emg_circuit_2_ext_amp #PWR3
 U 1 1 588ADF4E
 P 2450 7150
-F 0 "#PWR01" H 2450 7150 30  0001 C CNN
+F 0 "#PWR3" H 2450 7150 30  0001 C CNN
 F 1 "GND" H 2450 7080 30  0001 C CNN
 F 2 "" H 2450 7150 60  0000 C CNN
@@
 $EndComp
 $Comp
-L VCC #PWR02
+L VCC #PWR2
 U 1 1 588ADF4F
 P 2450 6700
-F 0 "#PWR02" H 2450 6800 30  0001 C CNN
+F 0 "#PWR2" H 2450 6800 30  0001 C CNN
 F 1 "VCC" H 2450 6800 30  0000 C CNN
 F 2 "" H 2450 6700 60  0000 C CNN
@@
 $EndComp
 $Comp
-L GND-RESCUE-emg_circuit_2_ext_amp #PWR03
+L GND-RESCUE-emg_circuit_2_ext_amp #PWR15
 U 1 1 589975BD
 P 13400 3250
-F 0 "#PWR03" H 13400 3250 30  0001 C CNN
+F 0 "#PWR15" H 13400 3250 30  0001 C CNN
 F 1 "GND" H 13400 3180 30  0001 C CNN
 F 2 "" H 13400 3250 60  0000 C CNN
@@
 $EndComp
 $Comp
-L VCC #PWR04
+L VCC #PWR1
 U 1 1 58A71443
 P 1100 7850
-F 0 "#PWR04" H 1100 7950 30  0001 C CNN
+F 0 "#PWR1" H 1100 7950 30  0001 C CNN
 F 1 "VCC" H 1100 7950 30  0000 C CNN
 F 2 "" H 1100 7850 60  0000 C CNN
@@
 Text Label 6800 7250 2    60   ~ 0
 IN2
-Text Label 6800 7450 2    60   ~ 0
+Text Label 6700 8050 2    60   ~ 0
 IN1
 Text Label 7000 6500 2    60   ~ 0
@@
 DGND
 $Comp
-L GND-RESCUE-emg_circuit_2_ext_amp #PWR05
+L GND-RESCUE-emg_circuit_2_ext_amp #PWR16
 U 1 1 58B4A72D
 P 13900 4050
-F 0 "#PWR05" H 13900 4050 30  0001 C CNN
+F 0 "#PWR16" H 13900 4050 30  0001 C CNN
 F 1 "GND" H 13900 3980 30  0001 C CNN
 F 2 "" H 13900 4050 60  0000 C CNN
@@
 Text Label 6800 7150 2    60   ~ 0
 IN2-
-Text Label 6800 7350 2    60   ~ 0
+Text Label 6700 7950 2    60   ~ 0
 IN1-
 $Comp
 L CONN_01X08 P5
 U 1 1 591A9761
-P 6100 7100
-F 0 "P5" H 6100 7550 50  0000 C CNN
-F 1 "CONN_01X08" V 6200 7100 50  0000 C CNN
-F 2 "Pin_Headers:Pin_Header_Straight_1x08_Pitch2.54mm" H 6100 7100 50  0001 C CNN
-F 3 "" H 6100 7100 50  0000 C CNN
-	1    6100 7100
+P 6000 7100
+F 0 "P5" H 6000 7550 50  0000 C CNN
+F 1 "CONN_01X08" V 6100 7100 50  0000 C CNN
+F 2 "Pin_Headers:Pin_Header_Straight_1x08_Pitch2.54mm" H 6000 7100 50  0001 C CNN
+F 3 "" H 6000 7100 50  0000 C CNN
+	1    6000 7100
 	-1   0    0    1
 $EndComp
@@
 $EndComp
 $Comp
-L GND-RESCUE-emg_circuit_2_ext_amp #PWR06
+L GND-RESCUE-emg_circuit_2_ext_amp #PWR9
 U 1 1 59BAC2D3
 P 7400 13350
-F 0 "#PWR06" H 7400 13350 30  0001 C CNN
+F 0 "#PWR9" H 7400 13350 30  0001 C CNN
 F 1 "GND" H 7400 13280 30  0001 C CNN
 F 2 "" H 7400 13350 60  0000 C CNN
@@
 $EndComp
 $Comp
-L GND-RESCUE-emg_circuit_2_ext_amp #PWR07
+L GND-RESCUE-emg_circuit_2_ext_amp #PWR13
 U 1 1 59BB14F7
 P 9400 12500
-F 0 "#PWR07" H 9400 12500 30  0001 C CNN
+F 0 "#PWR13" H 9400 12500 30  0001 C CNN
 F 1 "GND" H 9400 12430 30  0001 C CNN
 F 2 "" H 9400 12500 60  0000 C CNN
@@
 DVDD
 $Comp
-L GND-RESCUE-emg_circuit_2_ext_amp #PWR08
+L GND-RESCUE-emg_circuit_2_ext_amp #PWR12
 U 1 1 59BD03E3
 P 9050 15100
-F 0 "#PWR08" H 9050 15100 30  0001 C CNN
+F 0 "#PWR12" H 9050 15100 30  0001 C CNN
 F 1 "GND" H 9050 15030 30  0001 C CNN
 F 2 "" H 9050 15100 60  0000 C CNN
@@
 $EndComp
 $Comp
-L GND-RESCUE-emg_circuit_2_ext_amp #PWR09
+L GND-RESCUE-emg_circuit_2_ext_amp #PWR6
 U 1 1 59BD3A23
 P 5500 16000
-F 0 "#PWR09" H 5500 16000 30  0001 C CNN
+F 0 "#PWR6" H 5500 16000 30  0001 C CNN
 F 1 "GND" H 5500 15930 30  0001 C CNN
 F 2 "" H 5500 16000 60  0000 C CNN
@@
 $EndComp
 $Comp
-L GND-RESCUE-emg_circuit_2_ext_amp #PWR010
+L GND-RESCUE-emg_circuit_2_ext_amp #PWR7
 U 1 1 59BD4141
 P 5850 16500
-F 0 "#PWR010" H 5850 16500 30  0001 C CNN
+F 0 "#PWR7" H 5850 16500 30  0001 C CNN
 F 1 "GND" H 5850 16430 30  0001 C CNN
 F 2 "" H 5850 16500 60  0000 C CNN
@@
 $EndComp
 $Comp
-L GND-RESCUE-emg_circuit_2_ext_amp #PWR011
+L GND-RESCUE-emg_circuit_2_ext_amp #PWR10
 U 1 1 59BD468F
 P 8250 15950
-F 0 "#PWR011" H 8250 15950 30  0001 C CNN
+F 0 "#PWR10" H 8250 15950 30  0001 C CNN
 F 1 "GND" H 8250 15880 30  0001 C CNN
 F 2 "" H 8250 15950 60  0000 C CNN
@@
 $EndComp
 $Comp
-L GND-RESCUE-emg_circuit_2_ext_amp #PWR012
+L GND-RESCUE-emg_circuit_2_ext_amp #PWR14
 U 1 1 59BDE8C7
 P 10000 18950
-F 0 "#PWR012" H 10000 18950 30  0001 C CNN
+F 0 "#PWR14" H 10000 18950 30  0001 C CNN
 F 1 "GND" H 10000 18880 30  0001 C CNN
 F 2 "" H 10000 18950 60  0000 C CNN
@@
 GPIO_OVERCURRENT
 $Comp
-L GND-RESCUE-emg_circuit_2_ext_amp #PWR013
+L GND-RESCUE-emg_circuit_2_ext_amp #PWR11
 U 1 1 59BF02B5
 P 8450 19400
-F 0 "#PWR013" H 8450 19400 30  0001 C CNN
+F 0 "#PWR11" H 8450 19400 30  0001 C CNN
 F 1 "GND" H 8450 19330 30  0001 C CNN
 F 2 "" H 8450 19400 60  0000 C CNN
@@
 $EndComp
 $Comp
-L GND-RESCUE-emg_circuit_2_ext_amp #PWR014
+L GND-RESCUE-emg_circuit_2_ext_amp #PWR8
 U 1 1 59BF1B1A
 P 6650 19500
-F 0 "#PWR014" H 6650 19500 30  0001 C CNN
+F 0 "#PWR8" H 6650 19500 30  0001 C CNN
 F 1 "GND" H 6650 19430 30  0001 C CNN
 F 2 "" H 6650 19500 60  0000 C CNN
@@
 Text Label 23900 6450 0    60   ~ 0
 GPIO_OVERCURRENT
-Text Label 24100 6950 0    60   ~ 0
+Text Label 20850 5950 0    60   ~ 0
 GPIO_ISET
-Text Label 24200 6800 0    60   ~ 0
+Text Label 20850 5850 0    60   ~ 0
 GPIO_TTDM_BAT_EN
 Text GLabel 13900 3750 1    60   Input ~ 0
@@
 FOR RECHARGING: \nusing Amphenol FCI 10103594-0001LF
 $Comp
-L USB_OTG J1
+L USB_OTG-RESCUE-EEG_ADS1299_2 J1
 U 1 1 59BAF4BC
 P 3550 7050
@@
 N.C.
 $Comp
-L GND-RESCUE-emg_circuit_2_ext_amp #PWR015
+L GND-RESCUE-emg_circuit_2_ext_amp #PWR4
 U 1 1 59BB26FA
 P 4100 7700
-F 0 "#PWR015" H 4100 7700 30  0001 C CNN
+F 0 "#PWR4" H 4100 7700 30  0001 C CNN
 F 1 "GND" H 4100 7630 30  0001 C CNN
 F 2 "" H 4100 7700 60  0000 C CNN
@@
 	1    0    0    -1
 $EndComp
-Text Label 20850 5850 2    60   ~ 0
+Text Label 24300 3100 2    60   ~ 0
 LED2
-Text Label 20850 5950 2    60   ~ 0
+Text Label 24400 3150 0    60   ~ 0
 LED3
 $Comp
@@
 $EndComp
 $Comp
-L GND-RESCUE-emg_circuit_2_ext_amp #PWR016
+L GND-RESCUE-emg_circuit_2_ext_amp #PWR5
 U 1 1 59BE4F90
 P 4300 8700
-F 0 "#PWR016" H 4300 8700 30  0001 C CNN
+F 0 "#PWR5" H 4300 8700 30  0001 C CNN
 F 1 "GND" H 4300 8630 30  0001 C CNN
 F 2 "" H 4300 8700 60  0000 C CNN
@@
 Wire Wire Line
 	24200 5700 24200 6800
+Wire Wire Line
+	24200 3300 24200 3100
+Wire Wire Line
+	24200 3100 24300 3100
+Wire Wire Line
+	24300 3300 24300 3150
+Wire Wire Line
+	24300 3150 24400 3150
+$Comp
+L CONN_01X02 P7
+U 1 1 59C51B42
+P 6100 8000
+F 0 "P7" H 6100 8150 50  0000 C CNN
+F 1 "CONN_01X02" V 6200 8000 50  0000 C CNN
+F 2 "" H 6100 8000 50  0000 C CNN
+F 3 "" H 6100 8000 50  0000 C CNN
+	1    6100 8000
+	-1   0    0    1
+$EndComp
+Wire Wire Line
+	6300 7950 6700 7950
+Wire Wire Line
+	6300 8050 6700 8050
+$Comp
+L CONN_01X02 P8
+U 1 1 59C52C71
+P 6100 8500
+F 0 "P8" H 6100 8650 50  0000 C CNN
+F 1 "CONN_01X02" V 6200 8500 50  0000 C CNN
+F 2 "" H 6100 8500 50  0000 C CNN
+F 3 "" H 6100 8500 50  0000 C CNN
+	1    6100 8500
+	-1   0    0    1
+$EndComp
+Wire Wire Line
+	6300 8450 6650 8450
+Wire Wire Line
+	6300 8550 6650 8550
+Text Label 6650 8550 2    60   ~ 0
+IN2
+Text Label 6650 8450 2    60   ~ 0
+IN2-
+$Comp
+L CONN_01X02 P9
+U 1 1 59C536A5
+P 7250 7950
+F 0 "P9" H 7250 8100 50  0000 C CNN
+F 1 "CONN_01X02" V 7350 7950 50  0000 C CNN
+F 2 "" H 7250 7950 50  0000 C CNN
+F 3 "" H 7250 7950 50  0000 C CNN
+	1    7250 7950
+	-1   0    0    1
+$EndComp
+Text Label 7750 8000 2    60   ~ 0
+IN3
+Text Label 7750 7900 2    60   ~ 0
+IN3-
+Wire Wire Line
+	7750 7900 7450 7900
+Wire Wire Line
+	7750 8000 7450 8000
+$Comp
+L CONN_01X02 P10
+U 1 1 59C54141
+P 7250 8500
+F 0 "P10" H 7250 8650 50  0000 C CNN
+F 1 "CONN_01X02" V 7350 8500 50  0000 C CNN
+F 2 "" H 7250 8500 50  0000 C CNN
+F 3 "" H 7250 8500 50  0000 C CNN
+	1    7250 8500
+	-1   0    0    1
+$EndComp
+Wire Wire Line
+	7450 8450 7750 8450
+Wire Wire Line
+	7450 8550 7750 8550
+Text Label 7750 8550 2    60   ~ 0
+IN4
+Text Label 7750 8450 2    60   ~ 0
+IN4-
 $EndSCHEMATC

Commit message: Battery Management circuit. Requires revision to different ICs.
Parts:
- removed BT1: Battery_Cell, symbol Battery_Cell
- removed C38: 0.1uF, Capacitors_SMD:C_0402, symbol C
- removed J1: USB_OTG, symbol USB_OTG-RESCUE-EEG_ADS1299_2
- removed P5: CONN_01X08, Pin_Headers:Pin_Header_Straight_1x08_Pitch2.54mm, symbol CONN_01X08
- removed R13: 400Ω, Resistors_SMD:R_0402, symbol R
- removed U6: TPS61098x, BGA_custom_TI:WSON_6_1.5x1.5mm, symbol TPS61098x
- added J1: CONN_01X05, symbol CONN_01X05
- added U6: TPS63001, symbol TPS63001
- C39: value 10uF -> 22uF
- L7: value 4.7µH -> 2.20µH
Connections:
- net labels added: VCC_SW, VIN_TPS63001, VOUT_TPS63001
- net labels removed: BATT_VOLTAGE, N.C.
- wire segments 395 -> 384
- no-connect marks 17 -> 18
Other:
- note added: "THIS INDUCTOR IS 0402 (DIGIKEY)"
- note added: "This is a boost controller. Not what we wants :("
- note added: "VIN"
- note added: "Vout"
- note added: "We're *NOT* using TPS610981"
- note removed: "3.3V out"
- note removed: "Apparently supposed to be 3.3µH????\nSee TI forumns/ WEBENCH"
- note removed: "We're using TPS610981"
- moved on the sheet: C2, C39, L7, P6
