File: EEG_ADS1299_4.kicad_pcb (KiCad board)
At the start: 2 copper layers, 45.2 x 21.7 mm, 88 parts, among them IC1 ADS1299, P1 CONN_2, P2 CONN_2, P3 CONN_1, P4 CONN_1, P5 CONN_01X08, P6 CONN_2, U1 TPS2294x, U2 TPS61222, U3 NRF528XX-QFAA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

Commit message: Huge update. Rough draft of device with battery management.
Parts:
- removed the C13 at (273.2, 141.3)
- removed the C3 at (275.4, 143.1)
- removed the C37 at (294.9, 157.2)
- removed the L2 at (270.7, 142.7)
- removed the P6 at (268.0, 138.5)
- removed the U2 at (273.3, 142.9)
- added C13 (x2): 10uF, SM0402, F.Cu at (272.0, 144.1)
- added C2: 10uF, SM0402, F.Cu at (270.5, 140.2)
- added C3 (x2): 10uF, SM0402, F.Cu at (273.8, 142.0)
- added L2 (x2): 4.7µH, SM0603, F.Cu at (273.4, 146.6)
- added P1: CONN_2, PIN_ARRAY_2X1, F.Cu at (267.5, 134.9)
- added U2 (x2): TPS61222, TO_SOT_Packages_SMD:SOT-363_SC-70-6, F.Cu at (273.6, 144.0)
- C1, C38, C39, C40: footprint Capacitors_SMD:C_0402 -> SM0402
- C37: renamed from C2; value 10uF -> 1uF
- R13, R14, R15, R16, R17, R18, R21: footprint Resistors_SMD:R_0402 -> SM0402
- R19, R20: value 10k -> 1M
- moved U1 22.8 mm to (283.7, 145.5), turned to 180 degrees
- moved C1 22.5 mm to (285.1, 147.0)
- moved C39 21.5 mm to (267.7, 143.3), turned to 180 degrees
- moved R17 19.7 mm to (278.0, 140.6), turned to 90 degrees
- moved C38 19.7 mm to (267.8, 140.6), turned to 180 degrees
- moved L7 18.1 mm to (270.1, 142.8), turned to 270 degrees
- moved R15 17.4 mm to (280.7, 145.6), turned to 90 degrees
- moved U5 17.1 mm to (279.2, 143.2), turned to 90 degrees
- moved D2 16.6 mm to (280.1, 126.6), turned to 0 degrees
- moved R16 16.6 mm to (277.5, 144.3), turned to 270 degrees
- moved R21 16.5 mm to (285.7, 145.5), turned to 90 degrees
- moved D4 16.4 mm to (281.1, 142.9)
- moved U6 14.3 mm to (267.8, 141.9), turned to 180 degrees
- moved R18 13.3 mm to (276.4, 144.3), turned to 90 degrees
- moved R13 13.0 mm to (269.6, 141.2)
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- renumbered P1 to P6
Connections:
- C37 pad 1: VCC -> AVSS
- C37 pad 2: AVSS -> /DC+INPUT
- P6 pad 1: VCC -> /DC+INPUT
- U3 pad 11: /LED2 -> Net-(U3-Pad11)
- U3 pad 12: /LED3 -> Net-(U3-Pad12)
- U3 pad 21: Net-(U3-Pad21) -> /LED2
- U3 pad 27: Net-(U3-Pad27) -> /LED3
- U3 pad 4: /BATT_ADC_AIN -> /GPIO_TTDM_BAT_EN
- U3 pad 5: /GPIO_CTRL_PWR_ON -> /GPIO_ISET
- U3 pad 6: /GPIO_OVERCURRENT -> /GPIO_CTRL_PWR_ON
- U3 pad 7: Net-(U3-Pad7) -> /BATT_ADC_AIN
- U3 pad 8: /GPIO_ISET -> Net-(U3-Pad8)
- U3 pad 9: /GPIO_TTDM_BAT_EN -> Net-(U3-Pad9)
Routing:
- net VCC: track 5.02 -> 48.0 mm
- net AVSS: track 178.3 -> 217.4 mm, vias 9 -> 11
- net DVDD: track 65.5 -> 79.9 mm, vias 6 -> 7
- net Net-(D4-Pad2): track 0.00 -> 11.1 mm, vias 0 -> 2
- net /GPIO_CTRL_PWR_ON: track 0.00 -> 10.2 mm
- net /DC+INPUT: track 0.00 -> 9.31 mm, vias 0 -> 1
- net Net-(D3-Pad1): track 0.00 -> 8.88 mm
- net /BATT_ADC_AIN: track 0.00 -> 7.88 mm
- net /GPIO_TTDM_BAT_EN: track 0.00 -> 6.68 mm
- net /GPIO_ISET: track 0.00 -> 6.39 mm
- net Net-(C1-Pad1): track 0.00 -> 6.16 mm
- net Net-(D4-Pad1): track 0.00 -> 4.84 mm, vias 0 -> 2
- net AVDD: track 66.2 -> 69.2 mm
- net Net-(L7-Pad2): track 0.00 -> 2.75 mm
- net /LED3: track 7.23 -> 5.06 mm
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Other:
- board size 45.2 x 21.7 mm -> 45.2 x 23.2 mm

Commit message: Minor aestehtic changes to PCB. Almsot complete, requires final revision.
Routing:
- net AVSS: track 217.4 -> 215.7 mm
Other:
- board text added: "+Vin"
- board text added: "+Vin (4.5→5.5V)"
- board text added: "BAT"
- board text added: "USB CHG"
- board text removed: "VIN"
- board text removed: "→5.5V"
Changed lines of the file:
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@@
     (links 246)
     (no_connects 0)
-    (area 265.849999 125.449999 311.150001 147.250001)
+    (area 255.037143 122.157123 320.907143 148.740001)
     (thickness 1.6)
-    (drawings 40)
+    (drawings 42)
     (tracks 781)
     (zones 0)
@@
       (drillshape 0)
       (scaleselection 1)
-      (outputdirectory Gerber_nRF52_EEG/))
+      (outputdirectory Gerber_nRF52_EEG_wBM/))
   )
   (net 0 "")
@@
     (at 281.82 138.3)
     (attr smd)
-    (fp_text reference C22 (at -0.15 -1) (layer F.SilkS)
+    (fp_text reference C22 (at 0.06 1.12) (layer F.SilkS)
       (effects (font (size 0.508 0.4572) (thickness 0.1143)))
     )
@@
     )
   )
+  (gr_text "USB CHG" (at 268.81 144.18) (layer F.SilkS)
+    (effects (font (size 0.75 0.75) (thickness 0.1)))
+  )
+  (gr_text "+Vin (4.5→5.5V)" (at 272.66 147.73) (layer F.SilkS)
+    (effects (font (size 0.6 0.6) (thickness 0.1)))
+  )
+  (gr_text +Vin (at 269.41 136.28 90) (layer F.SilkS)
+    (effects (font (size 0.75 0.75) (thickness 0.1)))
+  )
+  (gr_text GND (at 267.31 147.71) (layer F.SilkS)
+    (effects (font (size 0.75 0.75) (thickness 0.1)))
+  )
   (gr_line (start 311.08 125.5) (end 311.1 125.5) (angle 90) (layer Edge.Cuts) (width 0.1))
   (gr_line (start 311.08 148.69) (end 311.08 125.5) (angle 90) (layer Edge.Cuts) (width 0.1))
@@
   (gr_line (start 265.9 125.5) (end 265.9 148.69) (angle 90) (layer Edge.Cuts) (width 0.1))
   (gr_circle (center 274.9475 142.7075) (end 274.8475 142.9075) (layer F.SilkS) (width 0.2))
-  (gr_text →5.5V (at 256.38 145.17) (layer F.SilkS)
-    (effects (font (size 0.6 0.6) (thickness 0.09)))
-  )
   (gr_text + (at 306.02 130.55) (layer F.SilkS)
     (effects (font (size 0.74 0.75) (thickness 0.1)))
@@
     (effects (font (size 0.7 0.7) (thickness 0.1)))
   )
-  (gr_text GND (at 259.985 137.655) (layer F.SilkS)
-    (effects (font (size 0.75 0.75) (thickness 0.1)))
-  )
-  (gr_text VIN (at 257.29 140.82) (layer F.SilkS)
+  (gr_text BAT (at 267.412 137.974) (layer F.SilkS)
     (effects (font (size 0.75 0.75) (thickness 0.1)))
   )
@@
   (segment (start 271.408 138.62) (end 271.408 137.59242) (width 0.152) (layer F.Cu) (net 11))
   (segment (start 271.408 137.59242) (end 271.73042 137.27) (width 0.152) (layer F.Cu) (net 11))
+  (segment (start 282.582 138.3) (end 282.582 138.942) (width 0.229) (layer F.Cu) (net 12))
+  (segment (start 283.42 138.8) (end 287.75 138.8) (width 0.229) (layer B.Cu) (net 12))
+  (segment (start 282.93 139.29) (end 283.42 138.8) (width 0.229) (layer B.Cu) (net 12))
+  (via (at 282.93 139.29) (size 0.508) (drill 0.3302) (layers F.Cu B.Cu) (net 12))
+  (segment (start 282.582 138.942) (end 282.93 139.29) (width 0.229) (layer F.Cu) (net 12))
   (via (at 279.17 143.24) (size 0.508) (drill 0.3302) (layers F.Cu B.Cu) (net 12))
   (segment (start 279.17 144.29) (end 279.17 143.24) (width 0.152) (layer F.Cu) (net 12))
@@
   (segment (start 280.72 146.01958) (end 279.92916 146.01958) (width 0.152) (layer F.Cu) (net 12))
   (segment (start 279.92916 146.01958) (end 279.79958 145.89) (width 0.152) (layer F.Cu) (net 12))
-  (segment (start 282.582 138.3) (end 282.582 137.542) (width 0.152) (layer F.Cu) (net 12))
-  (segment (start 283.84 138.8) (end 287.75 138.8) (width 0.229) (layer B.Cu) (net 12))
-  (segment (start 282.08 137.04) (end 283.84 138.8) (width 0.229) (layer B.Cu) (net 12))
-  (via (at 282.08 137.04) (size 0.508) (drill 0.3302) (layers F.Cu B.Cu) (net 12))
-  (segment (start 282.582 137.542) (end 282.08 137.04) (width 0.152) (layer F.Cu) (net 12))
   (segment (start 286.975 130.67458) (end 287.72458 130.67458) (width 0.152) (layer F.Cu) (net 12))
   (segment (start 287.72458 130.67458) (end 288.25 131.2) (width 0.152) (layer F.Cu) (net 12))

Commit message: Updated battery management design v2 complete.
Parts:
- removed L3: 15nH, SM0402
- removed L4: 10uH, SM0603
- C10, C22, C23: footprint SM0603 -> SM0402
- moved C23 1.74 mm to (273.0, 137.7), turned to 270 degrees
- moved C22 0.55 mm to (281.5, 137.9)
- moved C10 0.30 mm to (292.3, 127.4)
Routing:
- net Net-(U3-Pad47): track 3.92 -> 0.00 mm
- net Net-(L3-Pad1): track 1.48 -> 0.00 mm
- net DVDD: track 79.9 -> 79.3 mm
